Commit message: build on the car computer,fix small bug

File: src/bit_description/bit_robotcar/robots/ur5.urdf (robot description, URDF)
Before this commit: robot ur5, 9 links, 8 joints
Links:
- removed link world
- link car_link: geometry collision mesh filename=package://bit_robotcar/meshes/car_link.dae; visual mesh filename=package://bit_robotcar/meshes/car_link.dae
Joints:
- removed joint world_joint

Commit message: 修改了一些Launch文件，修改了红外采图方式
有请求时采图，无请求时停止

File: src/bit_description/bit_robotcar/robots/ur5.urdf (robot description, URDF)
Before this commit: robot ur5, 8 links, 7 joints
Links:
- added link ee_link; collision box size=0.01 0.01 0.01
Joints:
- added joint ee_fixed_joint: type fixed, parent wrist_3_link, child ee_link, origin xyz=0.0 0.0823 0.0 rpy=0.0 0.0 1.57079632679

Commit message: 在车上测试了抓两块砖，放两块砖到action
实现了砖块先放后取到堆栈，根据砖的数量执行任务，错误机制还没有完成

File: src/bit_description/bit_robotcar/robots/ur5.urdf (robot description, URDF)
Before this commit: robot ur5, 9 links, 8 joints
Links:
- removed link ee_link
- added link grasping_frame, mass 0.1879; visual mesh filename=package://bit_robotcar/meshes/ur5/visual/endEffector.dae
- added link world
- link car_link: geometry collision mesh filename=package://bit_robotcar/meshes/car_link.dae; visual mesh filename=package://bit_bit_robotcar/meshes/car_link.dae
Joints:
- removed joint ee_fixed_joint
- added joint grasping_frame_joint: type fixed, parent wrist_3_link, child grasping_frame, origin xyz=0 0.08725 0 rpy=0 0 0
- added joint world_joint: type fixed, parent world, child car_link, origin xyz=0.0 0.0 0.0 rpy=0.0 0.0 0.0

Commit message: 新增了bit_plan包用于蓝图读取与任务规划
修改了UR5末端模型，新增了相应的TF节点
串口检测到高度时发布TF消息

File: src/bit_description/bit_robotcar/robots/ur5.urdf (robot description, URDF)
Before this commit: robot ur5, 10 links, 9 joints
Links:
- removed link world
- added link magnet_link, mass 1.219; visual sphere radius=0.01
- added link tof_link, mass 0.1879; visual sphere radius=0.01
- added link zed_link, mass 0.1879; visual sphere radius=0.02
- link base_link: geometry collision mesh filename=package://robotcar/meshes/ur5/collision/base.stl; visual mesh filename=package://robotcar/meshes/ur5/visual/base.dae
- link car_link: geometry collision mesh filename=package://robotcar/meshes/car_link.dae; visual mesh filename=package://robotcar/meshes/car_link.dae
- link forearm_link: geometry collision mesh filename=package://robotcar/meshes/ur5/collision/forearm.stl; visual mesh filename=package://robotcar/meshes/ur5/visual/forearm.dae
- link shoulder_link: geometry collision mesh filename=package://robotcar/meshes/ur5/collision/shoulder.stl; visual mesh filename=package://robotcar/meshes/ur5/visual/shoulder.dae
- link upper_arm_link: geometry collision mesh filename=package://robotcar/meshes/ur5/collision/upperarm.stl; visual mesh filename=package://robotcar/meshes/ur5/visual/upperarm.dae
- link wrist_1_link: geometry collision mesh filename=package://robotcar/meshes/ur5/collision/wrist1.stl; visual mesh filename=package://robotcar/meshes/ur5/visual/wrist1.dae
- link wrist_2_link: geometry collision mesh filename=package://robotcar/meshes/ur5/collision/wrist2.stl; visual mesh filename=package://robotcar/meshes/ur5/visual/wrist2.dae
- link wrist_3_link: geometry collision mesh filename=package://robotcar/meshes/ur5/collision/wrist3.stl; visual mesh filename=package://robotcar/meshes/ur5/visual/wrist3.dae
Joints:
- removed joint world_joint
- added joint magnet_joint: type fixed, parent grasping_frame, child magnet_link, origin xyz=0.0 0.075 0.0 rpy=0.0 0.0 0.0
- added joint tof_joint: type fixed, parent wrist_3_link, child tof_link, origin xyz=0.01225 0.11125 0.0887  rpy=-1.5707963267948966 0.0 0.0
- added joint zed_joint: type fixed, parent wrist_3_link, child zed_link, origin xyz=-0.0235 0.10075 0.1424 rpy=-1.5707963267948966 0.0 0.0
- joint car_base_joint: type fixed -> prismatic
- joint shoulder_pan_joint: origin xyz=0.0 0.0 0.08 rpy=0.0 0.0 -1.57079632679 -> xyz=0.0 0.0 0.089159 rpy=0.0 0.0 0.0

Commit message: simple test in car

File: src/bit_description/bit_robotcar/robots/ur5.urdf (robot description, URDF)
Before this commit: robot ur5, 12 links, 11 joints
Joints:
- joint car_base_joint: origin xyz=0.448 0 0.615 rpy=0.0 0.0 0 -> xyz=0.448 0 0.615 rpy=0.0 0.0 -1.57079632679; type prismatic -> fixed
