Commit message: 修改了模型显示部分

File: src/bit_description/bit_robotcar/robots/ur5e.urdf (robot description, URDF)
Before this commit: robot ur5e, 12 links, 11 joints
Joints:
- joint car_base_joint: origin xyz=0.45 0 0.490 rpy=0.0 0.0 1.57079 -> xyz=0.45 0 0.490 rpy=0.0 0.0 0
- joint shoulder_pan_joint: origin xyz=0.0 0.0 0.163 rpy=0.0 0.0 -3.141593 -> xyz=0.0 0.0 0.163 rpy=0.0 0.0 0.0

Commit message: 修改模型的初始角度与安装状态一致

File: src/bit_description/bit_robotcar/robots/ur5e.urdf (robot description, URDF)
Before this commit: robot ur5e, 12 links, 11 joints
Joints:
- joint car_base_joint: origin xyz=0.45 0 0.490 rpy=0.0 0.0 0 -> xyz=0.45 0 0.490 rpy=0.0 0.0 1.57079
- joint shoulder_pan_joint: origin xyz=0.0 0.0 0.163 rpy=0.0 0.0 0.0 -> xyz=0.0 0.0 0.163 rpy=0.0 0.0 -3.141593

File: src/bit_description/bit_robotcar/robots/ur5e_challenge2.urdf (robot description, URDF)
Before this commit: robot ur5e, 11 links, 10 joints
Joints:
- joint car_base_joint: origin xyz=0.45 0 0.490 rpy=0.0 0.0 0 -> xyz=0.45 0 0.490 rpy=0.0 0.0 1.57079
- joint shoulder_pan_joint: origin xyz=0.0 0.0 0.163 rpy=0.0 0.0 0.0 -> xyz=0.0 0.0 0.163 rpy=0.0 0.0 -3.141593

File: src/bit_description/bit_robotcar/robots/ur5e_penzi.urdf (robot description, URDF)
Before this commit: robot ur5e, 11 links, 10 joints
Joints:
- joint car_base_joint: origin xyz=0.45 0 0.490 rpy=0.0 0.0 0 -> xyz=0.45 0 0.490 rpy=0.0 0.0 1.57079
- joint shoulder_pan_joint: origin xyz=0.0 0.0 0.163 rpy=0.0 0.0 0.0 -> xyz=0.0 0.0 0.163 rpy=0.0 0.0 -3.141593
