Commit message: 将砖块识别程序融入了系统

File: src/bit_description/bit_robotcar/robots/ur5e_challenge2.urdf (robot description, URDF)
Before this commit: robot ur5e, 11 links, 10 joints
Links:
- removed link gongye_camera_link
- added link MER_link, mass 1.219; visual sphere radius=0.01
Joints:
- removed joint gongye_camera_joint
- removed joint penzi_joint
- added joint MER_joint: type fixed, parent grasping_frame, child MER_link, origin xyz=0.0695 -0.022 0.143 rpy=-1.57079 0.0 0.0
- added joint zed_joint: type fixed, parent grasping_frame, child zed_link, origin xyz=-0.0465 0.0015 0.142  rpy=-1.57079 0.0 0.0

File: src/bit_description/bit_robotcar/robots/ur5e_challenge3.urdf (robot description, URDF)
Before this commit: robot ur5e, 11 links, 10 joints
Joints:
- joint infrared_joint: origin xyz=0.0 0.05147 0.077 rpy=0.0 0.0 0.0 -> xyz=0.0 0.05147 0.077 rpy=-1.57079 0.0 0.0
- joint penzi_joint: origin xyz=0.0 0.119 -0.0615  rpy=0 0.0 0.0 -> xyz=0.0 0.119 -0.0615  rpy=-1.57079 0.0 0.0

Commit message: 实现了工业相机矫正前图像的处理

File: src/bit_description/bit_robotcar/robots/ur5e_challenge2.urdf (robot description, URDF)
Before this commit: robot ur5e, 11 links, 10 joints
Joints:
- joint MER_joint: origin xyz=0.0695 -0.022 0.143 rpy=-1.57079 0.0 0.0 -> xyz=0.0695 0.0025628 0.143 rpy=-1.57079 0.0 0.0

Commit message: 调整TF
1、去掉ZED自己发布到TF信息
2、加上了zed_linkL和zed_linkR两个TF点
3、去掉了zed相机到屏幕显示

File: src/bit_description/bit_robotcar/robots/ur5e_challenge2.urdf (robot description, URDF)
Before this commit: robot ur5e, 11 links, 10 joints
Links:
- removed link zed_link
- added link zed_linkL, mass 0.1879; visual sphere radius=0.01
- added link zed_linkR, mass 0.1879; visual sphere radius=0.01
Joints:
- removed joint zed_joint
- added joint zed_jointL: type fixed, parent grasping_frame, child zed_linkL, origin xyz=-0.0465 0.0015 0.142  rpy=-1.57079 0.0 0.0
- added joint zed_jointR: type fixed, parent grasping_frame, child zed_linkR, origin xyz=0.0165 0.0015 0.142  rpy=-1.57079 0.0 0.0

Commit message: 校正grasping_frame位姿，为求解逆运动学

File: src/bit_description/bit_robotcar/robots/ur5e_challenge2.urdf (robot description, URDF)
Before this commit: robot ur5e, 12 links, 11 joints
Joints:
- joint MER_joint: origin xyz=0.0695 0.0025628 0.143 rpy=-1.57079 0.0 0.0 -> xyz=0.0695 -0.143 -0.0324372 rpy=0.0 0.0 0.0
- joint grasping_frame_joint: origin xyz=0 0.09237 0 rpy=0 0 0 -> xyz=0.0 0.12737 0.0 rpy=-1.570796 0 0
- joint zed_jointL: origin xyz=-0.0465 0.0015 0.142  rpy=-1.57079 0.0 0.0 -> xyz=-0.0465 -0.142 -0.0335  rpy=0.0 0.0 0.0
- joint zed_jointR: origin xyz=0.0165 0.0015 0.142  rpy=-1.57079 0.0 0.0 -> xyz=0.0165 -0.142 -0.0335  rpy=0.0 0.0 0.0

Commit message: 修改L架视觉检测

File: src/bit_description/bit_robotcar/robots/ur5e_challenge2.urdf (robot description, URDF)
Before this commit: robot ur5e, 12 links, 11 joints
Joints:
- joint car_base_joint: origin xyz=0.45 0 0.490 rpy=0.0 0.0 1.57079 -> xyz=0.45 0 0.365 rpy=0.0 0.0 1.57079
