Commit message: 修改ZED相机参数

File: src/zed_wrapper/urdf/zedm.urdf (robot description, URDF)
Before this commit: robot zedm_camera, 7 links, 6 joints
Links:
- removed link base_link
- added link zed_link
Joints:
- joint zed_camera_center_joint: origin xyz=0 0 0 rpy=0 0 0 -> xyz=0 0 0 rpy=0 -1.57079632679 1.57079632679; parent base_link -> zed_link
